File: cn3302.brd (EAGLE design)
At the start: 100 x 80 mm, 20 parts, among them M1 CN3302SOP-8

Commit message: pcb
Parts:
- moved R2 4.59 mm to (8.34, 4.61)
- moved C1 3.60 mm to (4.00, 24.4)
- moved C3 1.80 mm to (4.00, 22.2)
- moved C5 1.60 mm to (4.00, 17.6)
Routing:
- net 5V: track 0.00 -> 6.42 mm, vias 0 -> 3
- net N$5: track 0.00 -> 0.69 mm
Other:
- board size 100 x 80 mm -> 53 x 32 mm

Commit message: Проложил дорожки
Parts:
- moved C8 24.1 mm to (26.9, 16.7)
- moved C7 22.6 mm to (24.4, 16.7)
- moved C6 21.0 mm to (22.0, 16.7)
- moved C2 19.4 mm to (19.6, 16.7)
- moved VT2 14.3 mm to (15.3, 7.00), turned to 90 degrees
- moved D1 13.6 mm to (22.6, 7.10)
- moved D2 6.79 mm to (34.3, 24.9)
- moved L1 5.83 mm to (28.0, 25.0), turned to 270 degrees
- moved R3 5.46 mm to (16.9, 15.6)
- moved VT1 3.94 mm to (20.5, 26.2)
- moved RCS 3.44 mm to (11.5, 24.9)
- moved R2 3.32 mm to (6.04, 7.01)
- moved M1 2.28 mm to (13.0, 19.0)
- moved C1 2.00 mm to (4.00, 22.4)
- moved C3 2.00 mm to (4.00, 20.2)
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Connections:
- net GND: now also VT2.3; no longer VT2.1
- net N$10: now also VT2.2; no longer VT2.3
- net N$8: now also VT2.1; no longer VT2.2
Routing:
- net GND: track 0.00 -> 57.8 mm, vias 2 -> 6
- net N$10: track 0.00 -> 44.1 mm
- net 8.4V: track 0.00 -> 29.3 mm, vias 1 -> 5
- net N$9: track 0.00 -> 23.0 mm, vias 0 -> 2
- net N$5: track 0.69 -> 21.7 mm, vias 0 -> 2
- net 5V: track 6.42 -> 23.1 mm, vias 3 -> 1
- net N$6: track 0.00 -> 10.2 mm
- net N$1: track 0.10 -> 8.00 mm, vias 0 -> 1
- net N$3: track 0.00 -> 7.61 mm
- net N$2: track 0.00 -> 6.24 mm, vias 0 -> 1
- net N$8: track 0.00 -> 3.53 mm
- net N$4: track 0.00 -> 1.82 mm
Other:
- board size 53 x 32 mm -> 43 x 30 mm

Commit message: pcb
Parts:
- moved D1 19.6 mm to (27.7, 26.0)
- moved VT2 14.8 mm to (25.0, 18.1), turned to 180 degrees
- moved D2 6.99 mm to (33.0, 18.0)
- moved L1 5.34 mm to (33.2, 26.3)
- moved R3 4.23 mm to (19.2, 19.1), turned to 90 degrees
- moved C8 4.13 mm to (26.9, 12.6)
- moved C7 4.05 mm to (24.4, 12.7)
- moved C6 4.00 mm to (21.9, 12.7)
- moved C2 3.96 mm to (19.6, 12.7)
- moved C4 1.45 mm to (5.41, 17.6)
- moved C5 1.45 mm to (5.41, 15.4)
- moved C1 1.45 mm to (5.41, 22.1)
- moved C3 1.45 mm to (5.41, 19.9)
Routing:
- net N$10: track 44.1 -> 5.40 mm, vias 0 -> 1
- net GND: track 57.8 -> 35.1 mm, vias 6 -> 5
- net 8.4V: track 29.3 -> 22.5 mm, vias 5 -> 3
- net N$9: track 23.0 -> 16.7 mm, vias 2 -> 1
- net 5V: track 23.1 -> 18.6 mm
- net N$8: track 3.53 -> 0.00 mm
- net N$1: track 8.00 -> 5.08 mm
- net N$4: track 1.82 -> 3.84 mm
- net N$5: track 21.7 -> 21.1 mm
- added copper zone on layer 1, net GND
- added copper zone on layer 16, net GND
Other:
- board size 43 x 30 mm -> 44 x 31 mm
- board text added: "GND"
- board text added: "VIN"
