File: cn3302.brd (EAGLE design)
At the start: 44 x 23 mm, 20 parts, among them M1 CN3302SOP-8

Commit message: pcb
Parts:
- moved R3 3.67 mm to (23.4, 13.5), turned to 0 degrees
- moved D1 0.48 mm to (27.9, 17.9)
Routing:
- net GND: track 62.2 -> 96.4 mm, vias 6 -> 7
- net N$4: track 5.45 -> 2.47 mm
- net N$5: track 17.3 -> 15.0 mm
- net 5V: track 40.9 -> 39.6 mm
- net N$1: track 5.72 -> 4.43 mm
- net N$10: vias 0 -> 6
- added copper zone on layer 1, net N$10

Commit message: исправил плату
Parts:
- moved D2 10.9 mm to (45.2, 17.2)
- moved C8 10.9 mm to (27.9, 7.57), turned to 90 degrees
- moved C7 7.39 mm to (25.4, 7.65), turned to 90 degrees
- moved VT2 6.81 mm to (35.5, 7.90)
- moved L1 6.32 mm to (40.0, 16.4)
- moved M1 6.32 mm to (23.6, 12.7)
- moved R3 6.32 mm to (29.4, 11.5)
- moved VT1 6.32 mm to (25.9, 17.9)
- moved D1 6.32 mm to (33.9, 15.9)
- moved C1 5.39 mm to (9.85, 12.0)
- moved C3 5.39 mm to (9.85, 9.79)
- moved C4 5.39 mm to (9.85, 7.59)
- moved C5 5.39 mm to (9.85, 5.39)
- moved LED2 5.04 mm to (15.0, 14.0)
- moved LED1 4.84 mm to (15.0, 8.00)
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Routing:
- net GND: track 96.4 -> 161.7 mm, vias 7 -> 15
- net 8.4V: track 42.3 -> 68.9 mm
- net N$2: track 11.0 -> 18.4 mm
- net N$6: track 11.5 -> 13.5 mm
- net 5V: track 39.6 -> 37.8 mm
- net N$10: track 12.9 -> 14.6 mm, vias 6 -> 25
- net N$1: track 4.43 -> 3.42 mm
- net N$5: track 15.0 -> 15.6 mm
- added copper zone on layer 16, net N$10
Other:
- board size 44 x 23 mm -> 54 x 20 mm

Commit message: pcb
Parts:
- removed RCS: 0.015, 1_RESISTORS:2512
- added R4: 1.8, 1_RESISTORS:0603
- R3: value 1.8 -> 0.015; device 1_RESISTORS:0603 -> 1_RESISTORS:2512
- moved R3 16.6 mm to (14.5, 18.9)
- moved C5 10.8 mm to (20.4, 7.64), turned to 90 degrees
- moved C2 10.6 mm to (9.85, 7.59), turned to 0 degrees
- moved C1 6.60 mm to (9.85, 5.39)
- moved C4 4.40 mm to (9.85, 12.0)
- renumbered VT2 to T1
Connections:
- net 5V: now also C2.2, R3.1; no longer C5.2, RCS.1
- net 8.4V: now also C5.2; no longer C2.2
- net N$4: now also R4.1; no longer R3.1
- net N$6: now also R3.2; no longer RCS.2
- net N$8: now also R4.2; no longer R3.2
Routing:
- net N$10: track 14.6 -> 16.9 mm
- net GND: track 161.7 -> 163.4 mm
- net N$5: track 15.6 -> 14.6 mm
- net 8.4V: track 68.9 -> 69.5 mm

Commit message: Исправил плату
Parts:
- moved C1 1.00 mm to (10.8, 5.39)
- moved C2 1.00 mm to (10.8, 7.59)
- moved C3 1.00 mm to (10.8, 9.79)
- moved C4 1.00 mm to (10.8, 12.0)
- moved C5 1.00 mm to (21.4, 7.64)
- moved C6 1.00 mm to (23.9, 7.70)
- moved C7 1.00 mm to (26.4, 7.65)
- moved C8 1.00 mm to (28.9, 7.57)
- moved D1 1.00 mm to (34.9, 15.9)
- moved L1 1.00 mm to (41.0, 16.4)
- moved LED1 1.00 mm to (16.0, 8.00)
- moved LED2 1.00 mm to (16.0, 14.0)
- moved M1 1.00 mm to (24.6, 12.7)
- moved R1 1.00 mm to (14.2, 4.68)
- moved R2 1.00 mm to (17.2, 4.66)
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Routing:
- net 8.4V: track 69.5 -> 59.3 mm
- net N$2: track 18.4 -> 10.5 mm
- net GND: track 163.4 -> 158.0 mm
Other:
- outline, holes or cut-outs redrawn
