File: cn3302.brd (EAGLE design)
At the start: 56 x 20 mm, 20 parts, among them M1 CN3302SOP-8, T1 AOD9N50

Commit message: design block
Routing:
- net GND: track 156.4 -> 155.7 mm
Other:
- board text added: "VOUT"
Changed lines of the file:
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@@
 <drawing>
 <settings>
-<setting alwaysvectorfont="yes"/>
+<setting alwaysvectorfont="no"/>
 <setting verticaltext="up"/>
 </settings>
@@
 <wire x1="1" y1="4" x2="4" y2="1" width="0" layer="20" curve="90"/>
 <text x="19.66" y="18.63" size="1.778" layer="26" rot="MR0">CN3302</text>
+<text x="53.51" y="8.27" size="0.8128" layer="21">GND</text>
+<text x="53" y="12" size="0.8128" layer="25">VOUT</text>
 </plain>
 <attributes>
@@
 <wire x1="45.19" y1="9.08" x2="45.14" y2="9.13" width="0.6096" layer="1"/>
 <via x="10.573240625" y="12.013240625" extent="1-16" drill="0.35"/>
-<wire x1="12.00054375" y1="2.67" x2="20" y2="2.67" width="0.6096" layer="16"/>
 <wire x1="20" y1="2.67" x2="36" y2="2.67" width="0.6096" layer="16"/>
 <wire x1="36" y1="2.67" x2="46.67" y2="2.67" width="0.6096" layer="16"/>
@@
 <via x="9" y="16" extent="1-16" drill="0.35"/>
 <via x="31" y="9" extent="1-16" drill="0.35"/>
-<wire x1="5.72054375" y1="8.95" x2="4.15" y2="8.95" width="0.6096" layer="16"/>
-<wire x1="6" y1="8.93" x2="8.12" y2="8.93" width="0.6096" layer="16"/>
-<wire x1="5.72054375" y1="8.95" x2="12.00054375" y2="2.67" width="0.6096" layer="16"/>
-<wire x1="6" y1="7" x2="6" y2="8.93" width="0.6096" layer="16"/>
 <wire x1="9" y1="16" x2="9" y2="15.97" width="0.6096" layer="16"/>
 <wire x1="9" y1="15.97" x2="8" y2="14.97" width="0.6096" layer="16"/>
@@
 <wire x1="31" y1="9" x2="33.9848" y2="9" width="0.6096" layer="1"/>
 <wire x1="8" y1="12" x2="8.12" y2="11.88" width="0.6096" layer="16"/>
-<wire x1="8.12" y1="11.88" x2="8.12" y2="8.93" width="0.6096" layer="16"/>
 <wire x1="10.573240625" y1="12.013240625" x2="14.273240625" y2="12.013240625" width="0.6096" layer="16"/>
 <wire x1="14.273240625" y1="12.013240625" x2="14.72" y2="12.46" width="0.6096" layer="16"/>
@@
 </polygon>
 <via x="3" y="11" extent="1-16" drill="0.35"/>
-<wire x1="4.15" y1="8.95" x2="3" y2="10.1" width="0.6096" layer="16"/>
-<wire x1="3" y1="10.1" x2="3" y2="11" width="0.6096" layer="16"/>
 <via x="18.74" y="5.31" extent="1-16" drill="0.35"/>
 <via x="50" y="17" extent="1-16" drill="0.35"/>
@@
 <wire x1="20" y1="2" x2="18.74" y2="3.26" width="0.6096" layer="16"/>
 <wire x1="18.74" y1="3.26" x2="18.74" y2="5.31" width="0.6096" layer="16"/>
-<wire x1="5.72054375" y1="8.95" x2="6" y2="8.93" width="0" layer="19" extent="16-16"/>
+<wire x1="8" y1="12" x2="8" y2="9" width="0.6096" layer="16"/>
+<wire x1="8" y1="9" x2="6" y2="9" width="0.6096" layer="16"/>
+<wire x1="6" y1="9" x2="4" y2="9" width="0.6096" layer="16"/>
+<wire x1="4" y1="9" x2="3" y2="10" width="0.6096" layer="16"/>
+<wire x1="3" y1="10" x2="3" y2="11" width="0.6096" layer="16"/>
+<wire x1="10.33" y1="2.67" x2="6" y2="7" width="0.6096" layer="16"/>
+<wire x1="6" y1="7" x2="6" y2="9" width="0.6096" layer="16"/>
+<wire x1="20" y1="2.67" x2="10.33" y2="2.67" width="0.6096" layer="16"/>
 </signal>
 <signal name="N$5">
