File: 1.28TFT.brd (EAGLE design)
At the start: 12 parts, among them M1 LCD_FPCST

Commit message: fix
Parts:
- C4: value 10u -> 10uF
- R14: value 1k -> 1K
- moved R12 8.29 mm to (10.4, 17.4)
- moved R14 1.90 mm to (14.1, 9.40)
- moved R13 1.40 mm to (15.7, 9.27)
Connections:
- new net N$3: M1.9, R9.P$1
- net SCL: no longer M1.9, R9.P$1
Changed lines of the file:
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@@
 <drawing>
 <settings>
-<setting alwaysvectorfont="yes"/>
+<setting alwaysvectorfont="no"/>
 <setting verticaltext="up"/>
 </settings>
@@
 </autorouter>
 <elements>
-<element name="C4" library="LARS_409_R,C,L" package="0603" package3d_urn="urn:adsk.eagle:package:30551165/3" value="10u" x="7.493" y="14.478" smashed="yes" rot="R90">
+<element name="C4" library="LARS_409_R,C,L" package="0603" package3d_urn="urn:adsk.eagle:package:30551165/3" value="10uF" x="7.493" y="14.478" smashed="yes" rot="R90">
 <attribute name="NAME" x="6.793" y="13.078" size="0.6" layer="25" font="vector" rot="R90"/>
 <attribute name="VALUE" x="8.793" y="12.878" size="0.6" layer="27" font="vector" rot="R90"/>
@@
 <attribute name="VALUE" x="6.066" y="10.998" size="0.6" layer="27" font="vector" rot="R270"/>
 </element>
-<element name="R12" library="LARS_409_R,C,L" package="0603" package3d_urn="urn:adsk.eagle:package:30551165/3" value="1k" x="12.573" y="9.398" smashed="yes" rot="R270">
-<attribute name="NAME" x="13.273" y="10.798" size="0.6" layer="25" font="vector" rot="R270"/>
-<attribute name="VALUE" x="11.273" y="10.998" size="0.6" layer="27" font="vector" rot="R270"/>
-</element>
-<element name="R13" library="LARS_409_R,C,L" package="0603" package3d_urn="urn:adsk.eagle:package:30551165/3" value="1k" x="14.351" y="9.398" smashed="yes" rot="R270">
-<attribute name="NAME" x="15.051" y="10.798" size="0.6" layer="25" font="vector" rot="R270"/>
-<attribute name="VALUE" x="13.051" y="10.998" size="0.6" layer="27" font="vector" rot="R270"/>
-</element>
-<element name="R14" library="LARS_409_R,C,L" package="0603" package3d_urn="urn:adsk.eagle:package:30551165/3" value="1k" x="16.002" y="9.398" smashed="yes" rot="R270">
-<attribute name="NAME" x="16.702" y="10.798" size="0.6" layer="25" font="vector" rot="R270"/>
-<attribute name="VALUE" x="14.702" y="10.998" size="0.6" layer="27" font="vector" rot="R270"/>
+<element name="R12" library="LARS_409_R,C,L" package="0603" package3d_urn="urn:adsk.eagle:package:30551165/3" value="1k" x="10.414" y="17.399" smashed="yes" rot="R270">
+<attribute name="NAME" x="11.114" y="18.799" size="0.6" layer="25" font="vector" rot="R270"/>
+<attribute name="VALUE" x="9.114" y="18.999" size="0.6" layer="27" font="vector" rot="R270"/>
+</element>
+<element name="R13" library="LARS_409_R,C,L" package="0603" package3d_urn="urn:adsk.eagle:package:30551165/3" value="1k" x="15.748" y="9.271" smashed="yes" rot="R270">
+<attribute name="NAME" x="16.448" y="10.671" size="0.6" layer="25" font="vector" rot="R270"/>
+<attribute name="VALUE" x="14.448" y="10.871" size="0.6" layer="27" font="vector" rot="R270"/>
+</element>
+<element name="R14" library="LARS_409_R,C,L" package="0603" package3d_urn="urn:adsk.eagle:package:30551165/3" value="1K" x="14.097" y="9.398" smashed="yes" rot="R270">
+<attribute name="NAME" x="14.797" y="10.798" size="0.6" layer="25" font="vector" rot="R270"/>
+<attribute name="VALUE" x="12.797" y="10.998" size="0.6" layer="27" font="vector" rot="R270"/>
 </element>
 <element name="R6" library="LARS_409_R,C,L" package="0603" package3d_urn="urn:adsk.eagle:package:30551165/3" value="2R" x="14.732" y="17.526" smashed="yes" rot="R180">
@@
 <contactref element="R13" pad="P$1"/>
 <wire x1="15.494" y1="13.524" x2="9.872" y2="20.998" width="0" layer="19" extent="1-1"/>
-<wire x1="14.351" y1="10.225" x2="15.494" y2="13.524" width="0" layer="19" extent="1-1"/>
+<wire x1="15.748" y1="10.098" x2="15.494" y2="13.524" width="0" layer="19" extent="1-1"/>
 </signal>
 <signal name="3.3V">
@@
 <contactref element="C6" pad="P$1"/>
 <contactref element="M1" pad="3"/>
-<via x="5.588" y="4.572" extent="1-16" drill="0.35"/>
-<wire x1="13.372" y1="20.998" x2="12.672" y2="20.998" width="0" layer="19" extent="1-1"/>
+<wire x1="12.672" y1="20.998" x2="13.372" y2="20.998" width="0" layer="19" extent="1-1"/>
 <wire x1="7.493" y1="13.651" x2="12.672" y2="20.998" width="0" layer="19" extent="1-1"/>
 <wire x1="5.461" y1="13.651" x2="7.493" y2="13.651" width="0" layer="19" extent="1-1"/>
 <wire x1="7.366" y1="8.571" x2="7.493" y2="13.651" width="0" layer="19" extent="1-1"/>
-<wire x1="5.588" y1="4.572" x2="7.366" y2="8.571" width="0" layer="19" extent="1-1"/>
 </signal>
 <signal name="GND">
 <contactref element="R6" pad="P$1"/>
-<contactref element="R8" pad="P$1"/>
 <contactref element="M1" pad="1"/>
 <contactref element="M1" pad="5"/>
@@
 <contactref element="C6" pad="P$2"/>
 <contactref element="C7" pad="P$2"/>
-<via x="7.366" y="4.572" extent="1-16" drill="0.35"/>
+<contactref element="R8" pad="P$1"/>
 <wire x1="11.972" y1="20.998" x2="14.772" y2="20.998" width="0" layer="19" extent="1-1"/>
 <wire x1="11.272" y1="20.998" x2="11.972" y2="20.998" width="0" layer="19" extent="1-1"/>
@@
 <wire x1="13.335" y1="15.178" x2="15.494" y2="15.178" width="0" layer="19" extent="1-1"/>
 <wire x1="7.072" y1="20.998" x2="11.272" y2="20.998" width="0" layer="19" extent="1-1"/>
-<wire x1="7.493" y1="15.305" x2="13.335" y2="15.178" width="0" layer="19" extent="1-1"/>
+<wire x1="7.493" y1="15.305" x2="7.072" y2="20.998" width="0" layer="19" extent="1-1"/>
 <wire x1="5.461" y1="15.305" x2="7.493" y2="15.305" width="0" layer="19" extent="1-1"/>
-<wire x1="7.366" y1="4.572" x2="7.493" y2="15.305" width="0" layer="19" extent="1-1"/>
 </signal>
 <signal name="D/C">
 <contactref element="R12" pad="P$2"/>
-<via x="12.573" y="4.572" extent="1-16" drill="0.35"/>
-<wire x1="12.573" y1="4.572" x2="12.573" y2="8.571" width="0" layer="19" extent="1-1"/>
 </signal>
 <signal name="CS">
 <contactref element="R13" pad="P$2"/>
-<via x="14.351" y="4.572" extent="1-16" drill="0.35"/>
-<wire x1="14.351" y1="4.572" x2="14.351" y2="8.571" width="0" layer="19" extent="1-1"/>
 </signal>
 <signal name="RST">
@@
 <contactref element="R14" pad="P$1"/>
 <wire x1="13.335" y1="13.524" x2="7.772" y2="20.998" width="0" layer="19" extent="1-1"/>
-<wire x1="16.002" y1="10.225" x2="13.335" y2="13.524" width="0" layer="19" extent="1-1"/>
+<wire x1="14.097" y1="10.225" x2="13.335" y2="13.524" width="0" layer="19" extent="1-1"/>
 <wire x1="7.366" y1="10.225" x2="13.335" y2="13.524" width="0" layer="19" extent="1-1"/>
 </signal>
@@
 <contactref element="R10" pad="P$1"/>
 <contactref element="R10" pad="P$2"/>
-<via x="10.795" y="4.572" extent="1-16" drill="0.35"/>
 <wire x1="10.795" y1="10.225" x2="8.472" y2="20.998" width="0" layer="19" extent="1-1"/>
 <wire x1="10.795" y1="8.571" x2="10.795" y2="10.225" width="0" layer="19" extent="1-1"/>
-<wire x1="10.795" y1="4.572" x2="10.795" y2="8.571" width="0" layer="19" extent="1-1"/>
 </signal>
 <signal name="SCL">
-<contactref element="M1" pad="9"/>
-<contactref element="R9" pad="P$1"/>
 <contactref element="R9" pad="P$2"/>
-<via x="9.144" y="4.572" extent="1-16" drill="0.35"/>
-<wire x1="9.144" y1="10.225" x2="9.172" y2="20.998" width="0" layer="19" extent="1-1"/>
-<wire x1="9.144" y1="8.571" x2="9.144" y2="10.225" width="0" layer="19" extent="1-1"/>
-<wire x1="9.144" y1="4.572" x2="9.144" y2="8.571" width="0" layer="19" extent="1-1"/>
 </signal>
 <signal name="DC">
 <contactref element="R12" pad="P$1"/>
 <contactref element="M1" pad="7"/>
-<wire x1="12.573" y1="10.225" x2="10.572" y2="20.998" width="0" layer="19" extent="1-1"/>
+<wire x1="10.414" y1="18.226" x2="10.572" y2="20.998" width="0" layer="19" extent="1-1"/>
 </signal>
 <signal name="RESET">
 <contactref element="R14" pad="P$2"/>
-<via x="16.002" y="4.572" extent="1-16" drill="0.35"/>
-<wire x1="16.002" y1="4.572" x2="16.002" y2="8.571" width="0" layer="19" extent="1-1"/>
+</signal>
+<signal name="N$3">
+<contactref element="R9" pad="P$1"/>
+<contactref element="M1" pad="9"/>
+<wire x1="9.144" y1="10.225" x2="9.172" y2="20.998" width="0" layer="19" extent="1-1"/>
 </signal>
 </signals>

Commit message: bugfix
Parts:
- C6, C7: value 0.1u -> 0.1uF
- R10, R12, R13, R9: value 1k -> 1K
- R11: value 10k -> 10K
- R8: value 51k -> 51K
- moved R14 11.6 mm to (5.59, 17.3)
- moved C7 10.2 mm to (3.56, 17.3), turned to 270 degrees
- moved R10 8.54 mm to (7.49, 17.3)
- moved R9 7.88 mm to (9.53, 17.3)
- moved R13 5.41 mm to (14.9, 14.6), turned to 0 degrees
- moved C4 2.98 mm to (5.59, 12.2)
- moved C6 2.98 mm to (3.56, 12.2)
- moved R11 2.80 mm to (7.49, 12.2)
- moved R8 2.37 mm to (14.9, 16.6), turned to 180 degrees
- moved R6 1.15 mm to (14.9, 18.7)
- moved R12 1.02 mm to (11.4, 17.3)
Connections:
- net DC renamed N$5
- new net N$4: M1.10, R10.P$1
- net SDA: no longer M1.10, R10.P$1
