File: cn3302 JLCPCB.brd (EAGLE design)
At the start: 54 x 20 mm, 20 parts, among them M1 CN3302SOP-8, T1 AOD9N50

Commit message: футпринт lid
Parts:
- moved C5 25.6 mm to (46.7, 12.0), turned to 0 degrees
- moved C6 22.7 mm to (46.6, 9.13), turned to 0 degrees
- moved C7 20.2 mm to (46.6, 6.18), turned to 0 degrees
- moved C8 18.2 mm to (46.7, 3.42), turned to 0 degrees
- moved M1 8.01 mm to (24.6, 4.68)
- moved D1 7.88 mm to (27.1, 17.1), turned to 0 degrees
- moved VT1 7.72 mm to (24.6, 10.6)
- moved R2 5.27 mm to (19.6, 9.37), turned to 90 degrees
- moved R4 3.88 mm to (29.8, 7.67), turned to 90 degrees
- moved L1 3.57 mm to (37.6, 17.6), turned to 0 degrees
- moved C1 2.28 mm to (10.9, 3.11)
- moved R1 1.94 mm to (14.2, 2.74), turned to 90 degrees
- moved R3 1.85 mm to (15.2, 17.1)
- moved C2 1.60 mm to (10.9, 5.99)
- moved LED2 1.54 mm to (16.0, 12.5), turned to 0 degrees
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Routing:
- net 8.4V: track 59.3 -> 45.3 mm
- net N$5: track 14.6 -> 7.85 mm, vias 2 -> 1
- net N$2: track 10.5 -> 4.33 mm
- net N$9: track 16.4 -> 20.9 mm, vias 0 -> 2
- net N$6: track 13.5 -> 16.9 mm
- net N$4: track 2.47 -> 5.87 mm
- net N$3: track 6.86 -> 9.89 mm
- net N$1: track 3.42 -> 5.36 mm
- net N$8: track 1.43 -> 2.92 mm
- net S$1: track 0.00 -> 0.90 mm, vias 0 -> 1
- net N$10: track 16.7 -> 17.3 mm
- net GND: track 157.8 -> 157.4 mm, vias 15 -> 11
Other:
- board size 54 x 20 mm -> 56 x 20 mm

Commit message: добавил word
Routing:
- net GND: track 157.4 -> 155.7 mm, vias 11 -> 12
- net S$1: track 0.90 -> 0.00 mm, vias 1 -> 0
Other:
- board text added: "VOUT"
Changed lines of the file:
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@@
 <wire x1="1" y1="4" x2="4" y2="1" width="0" layer="20" curve="90"/>
 <text x="19.66" y="18.63" size="1.778" layer="26" rot="MR0">CN3302</text>
+<text x="53.51" y="8.27" size="0.8128" layer="21">GND</text>
+<text x="53" y="12" size="0.8128" layer="25">VOUT</text>
 </plain>
 <attributes>
@@
 <contactref element="R4" pad="2"/>
 <contactref element="T1" pad="1"/>
-<wire x1="30.65628125" y1="9.8298" x2="30.8298" y2="9.8298" width="0.6096" layer="1"/>
-<wire x1="30.8298" y1="9.8298" x2="31" y2="10" width="0.6096" layer="1"/>
 <wire x1="29.76" y1="8.42" x2="29.76" y2="8.93351875" width="0.6096" layer="1"/>
-<wire x1="29.76" y1="8.93351875" x2="30.65628125" y2="9.8298" width="0.6096" layer="1"/>
-<wire x1="31.41" y1="10.186" x2="31.0538" y2="9.8298" width="0.1524" layer="1"/>
-<wire x1="31.0538" y1="9.8298" x2="30.8298" y2="9.8298" width="0.1524" layer="1"/>
+<wire x1="29.76" y1="8.93351875" x2="31.01248125" y2="10.186" width="0.6096" layer="1"/>
+<wire x1="31.01248125" y1="10.186" x2="31.41" y2="10.186" width="0.6096" layer="1"/>
 </signal>
 <signal name="N$9">
@@
 <wire x1="48.14" y1="9.13" x2="48.19" y2="9.18" width="0.6096" layer="1"/>
 <wire x1="48.14" y1="9.13" x2="48.14" y2="6.17" width="0.6096" layer="1"/>
-<wire x1="48.08" y1="3.51" x2="48.08" y2="6.18" width="0.6096" layer="1"/>
+<wire x1="48.17" y1="3.42" x2="48.08" y2="3.51" width="0.6096" layer="1"/>
+<wire x1="48.08" y1="6.18" x2="48.08" y2="3.51" width="0.6096" layer="1"/>
 <wire x1="51" y1="13" x2="50.02" y2="12.02" width="0.6096" layer="1"/>
 <wire x1="50.02" y1="12.02" x2="48.19" y2="12.02" width="0.6096" layer="1"/>
@@
 <wire x1="21.69" y1="4.045" x2="23.78148125" y2="4.045" width="0.6096" layer="1"/>
 <wire x1="23.78148125" y1="4.045" x2="26.12168125" y2="1.7048" width="0.6096" layer="1"/>
-<wire x1="47.7048" y1="1.7048" x2="48" y2="2" width="0.6096" layer="1"/>
-<wire x1="48" y1="3" x2="48" y2="2" width="0.6096" layer="1"/>
 <wire x1="26.12168125" y1="1.7048" x2="47.7048" y2="1.7048" width="0.6096" layer="1"/>
-<wire x1="48.17" y1="3.42" x2="48.08" y2="3.51" width="0.6096" layer="1"/>
-<wire x1="48.17" y1="3.42" x2="48.17" y2="3.17" width="0.6096" layer="1"/>
-<wire x1="48.17" y1="3.17" x2="48" y2="3" width="0.6096" layer="1"/>
-</signal>
-<signal name="S$1">
-<via x="3" y="11" extent="1-16" drill="0.35"/>
-<wire x1="3" y1="11" x2="3" y2="10.1" width="0.6096" layer="16"/>
+<wire x1="48.17" y1="2.17" x2="48.17" y2="3.42" width="0.6096" layer="1"/>
+<wire x1="47.7048" y1="1.7048" x2="48.17" y2="2.17" width="0.6096" layer="1"/>
 </signal>
 <signal name="GND">
@@
 <wire x1="45.19" y1="9.08" x2="45.14" y2="9.13" width="0.6096" layer="1"/>
 <via x="10.573240625" y="12.013240625" extent="1-16" drill="0.35"/>
-<wire x1="12.00054375" y1="2.67" x2="20" y2="2.67" width="0.6096" layer="16"/>
 <wire x1="20" y1="2.67" x2="36" y2="2.67" width="0.6096" layer="16"/>
 <wire x1="36" y1="2.67" x2="46.67" y2="2.67" width="0.6096" layer="16"/>
@@
 <via x="9" y="16" extent="1-16" drill="0.35"/>
 <via x="31" y="9" extent="1-16" drill="0.35"/>
-<wire x1="5.72054375" y1="8.95" x2="4.15" y2="8.95" width="0.6096" layer="16"/>
-<wire x1="6" y1="8.93" x2="8.12" y2="8.93" width="0.6096" layer="16"/>
-<wire x1="5.72054375" y1="8.95" x2="12.00054375" y2="2.67" width="0.6096" layer="16"/>
-<wire x1="6" y1="7" x2="6" y2="8.93" width="0.6096" layer="16"/>
 <wire x1="9" y1="16" x2="9" y2="15.97" width="0.6096" layer="16"/>
 <wire x1="9" y1="15.97" x2="8" y2="14.97" width="0.6096" layer="16"/>
@@
 <wire x1="31" y1="9" x2="33.9848" y2="9" width="0.6096" layer="1"/>
 <wire x1="8" y1="12" x2="8.12" y2="11.88" width="0.6096" layer="16"/>
-<wire x1="8.12" y1="11.88" x2="8.12" y2="8.93" width="0.6096" layer="16"/>
 <wire x1="10.573240625" y1="12.013240625" x2="14.273240625" y2="12.013240625" width="0.6096" layer="16"/>
 <wire x1="14.273240625" y1="12.013240625" x2="14.72" y2="12.46" width="0.6096" layer="16"/>
@@
 <vertex x="58" y="0"/>
 </polygon>
+<via x="3" y="11" extent="1-16" drill="0.35"/>
 <via x="18.74" y="5.31" extent="1-16" drill="0.35"/>
 <via x="50" y="17" extent="1-16" drill="0.35"/>
@@
 <wire x1="20" y1="2" x2="18.74" y2="3.26" width="0.6096" layer="16"/>
 <wire x1="18.74" y1="3.26" x2="18.74" y2="5.31" width="0.6096" layer="16"/>
-<wire x1="4.15" y1="8.95" x2="4.17" y2="8.93" width="0.6096" layer="16"/>
-<wire x1="4.17" y1="8.93" x2="6" y2="8.93" width="0.6096" layer="16"/>
-<wire x1="4.15" y1="8.95" x2="4.05" y2="8.95" width="0.6096" layer="16"/>
-<wire x1="4.05" y1="8.95" x2="3" y2="10" width="0.6096" layer="16"/>
+<wire x1="8" y1="12" x2="8" y2="9" width="0.6096" layer="16"/>
+<wire x1="8" y1="9" x2="6" y2="9" width="0.6096" layer="16"/>
+<wire x1="6" y1="9" x2="4" y2="9" width="0.6096" layer="16"/>
+<wire x1="4" y1="9" x2="3" y2="10" width="0.6096" layer="16"/>
+<wire x1="3" y1="10" x2="3" y2="11" width="0.6096" layer="16"/>
+<wire x1="10.33" y1="2.67" x2="6" y2="7" width="0.6096" layer="16"/>
+<wire x1="6" y1="7" x2="6" y2="9" width="0.6096" layer="16"/>
+<wire x1="20" y1="2.67" x2="10.33" y2="2.67" width="0.6096" layer="16"/>
 </signal>
 <signal name="N$5">
